Commit message: adapt tube code to latest moveit

File: config/ur5.ros2_control.xacro (robot description, xacro)
@@ -4,8 +4,16 @@
         <xacro:property name="initial_positions" value="${load_yaml(initial_positions_file)['initial_positions']}"/>
         <ros2_control name="${name}" type="system">
-            <hardware>
-                <!-- By default, set up controllers for simulation. This won't work on real hardware -->
-                <plugin>mock_components/GenericSystem</plugin>
-            </hardware>
+            <xacro:if value="${name == 'FakeSystem'}">
+                <hardware>
+                    <plugin>mock_components/GenericSystem</plugin>
+                </hardware>
+            </xacro:if>
+            <xacro:unless value="${name == 'FakeSystem'}">
+                <hardware>
+                    <plugin>topic_based_ros2_control/TopicBasedSystem</plugin>
+                    <param name="joint_commands_topic">/isaac_joint_commands</param>
+                    <param name="joint_states_topic">/isaac_joint_states</param>
+                </hardware>
+            </xacro:unless>
             <joint name="shoulder_pan_joint">
                 <command_interface name="position"/>
@@ -50,4 +58,10 @@
                 <state_interface name="velocity"/>
             </joint>
+            <joint name="robotiq_85_left_knuckle_joint">
+                <command_interface name="position"/>
+                <state_interface name="position">
+                </state_interface>
+                <state_interface name="velocity"/>
+            </joint>
         </ros2_control>
     </xacro:macro>
